File: kicad/whaleticker/whaleticker.kicad_pcb (KiCad board)
At the start: 2 copper layers, 35 x 34 mm, 24 parts, among them J1 USB_B_Micro, Q1 S8050_J3Y, Q2 PMBT2222AYS, U1 ESP-12E, U2 CP2102-GMR_NRND, U3 BL8565

Commit message: Changed PCB to WhaleTicker
Parts:
- removed QR*****: https://barn53.github.io/CoinThing/, https:__barn53.github.io_CoinThing_
- added G***: LOGO, Logo:LogoSmall, F.Cu at (159.1, 61.6)
- added G***: LOGO, Logo:Logo, B.Cu at (165.9, 79.2)
Other:
- board text added: "WhaleTicker rev.A 12/21"
- board text removed: "CoinThing"
- board text removed: "CoinThing a coin ticker display"
- board text removed: "CoinThing barn53 rev.E 05/21"
